Commit message: various tweaks

File: description/imu.xacro (robot description, xacro)
@@ -4,5 +4,5 @@
         <parent link="chassis"/>
         <child link="bno055"/>
-        <origin xyz="0 0 0.2" rpy="0 0 0"/>
+        <origin xyz="0 0 0.2" rpy="0 0 -1.5708"/>
     </joint>
     <link name="bno055">

Commit message: changes and new imu config

File: description/imu.xacro (robot description, xacro)
@@ -3,8 +3,8 @@
     <joint name="imu_joint" type="fixed">
         <parent link="chassis"/>
-        <child link="bno055"/>
-        <origin xyz="0 0 0.2" rpy="0 0 -1.5708"/>
+        <child link="imu_frame"/>
+        <origin xyz="0 0 0.2" rpy="0 1.5708 -1.5708"/>
     </joint>
-    <link name="bno055">
+    <link name="imu_frame">
         <visual>
             <geometry>
