Commit message: urdf tweaks

File: description/camera.xacro (robot description, xacro)
@@ -4,5 +4,5 @@
         <parent link="chassis"/>
         <child link="camera_link"/>
-        <origin xyz="0.276 0 0.181" rpy="0 0 0"/>
+        <origin xyz="0.05 0 0.23" rpy="0 0 0"/>
     </joint>
     <link name="camera_link">
@@ -14,5 +14,5 @@
         </visual>
         <visual>
-            <origin xyz="0 0 -0.05"/>
+            <origin xyz="0 0 0"/>
             <geometry>
                 <cylinder radius="0.002" length="0.1"/>

File: description/robot.urdf.xacro (robot description, xacro)
@@ -12,5 +12,5 @@
     <xacro:include filename="lidar.xacro" />
     <!-- <xacro:include filename="imu.xacro" /> -->
-    <!-- <xacro:include filename="camera.xacro" /> -->
+    <xacro:include filename="camera.xacro" />
     <!-- <xacro:include filename="depth_camera.xacro" /> -->
     <!-- <xacro:include filename="face.xacro" /> -->
