Commit message: sasas

File: description/robot_core.xacro (robot description, xacro)
@@ -52,5 +52,5 @@
             <origin xyz="${chassis_length/2} 0 ${chassis_height/2}"/>
             <geometry>
-                <box size="${chassis_length} ${chassis_width} ${chassis_height}"/>
+                <mesh filename="package://articubot_one/meshes/gazebo_turt_body.stl" scale="0.001 0.001 0.001"/>
             </geometry>
             <material name="orange"/>

Commit message: erre

File: description/robot_core.xacro (robot description, xacro)
@@ -52,5 +52,5 @@
             <origin xyz="${chassis_length/2} 0 ${chassis_height/2}"/>
             <geometry>
-                <mesh filename="package://articubot_one/meshes/gazebo_turt_body.stl" scale="0.001 0.001 0.001"/>
+                <mesh filename="package://articubot_one/meshes/gazebo_turt_body_adj.stl" scale="0.001 0.001 0.001"/>
             </geometry>
             <material name="orange"/>

Commit message: dffdf

File: description/robot_core.xacro (robot description, xacro)
@@ -52,5 +52,5 @@
             <origin xyz="${chassis_length/2} 0 ${chassis_height/2}"/>
             <geometry>
-                <mesh filename="package://articubot_one/meshes/gazebo_turt_body_adj.stl" scale="0.001 0.001 0.001"/>
+                <mesh filename="package://articubot_one/meshes/gazebo_turt_body.dae" scale="0.001 0.001 0.001"/>
             </geometry>
             <material name="orange"/>

Commit message: weweew

File: description/robot_core.xacro (robot description, xacro)
@@ -52,5 +52,5 @@
             <origin xyz="${chassis_length/2} 0 ${chassis_height/2}"/>
             <geometry>
-                <mesh filename="package://articubot_one/meshes/gazebo_turt_body.dae" scale="0.001 0.001 0.001"/>
+                <mesh filename="package://articubot_one/meshes/gazebo_turt_body.dae" scale="1 1 1"/>
             </geometry>
             <material name="orange"/>

Commit message: sfrtgedg

File: description/robot_core.xacro (robot description, xacro)
@@ -52,5 +52,5 @@
             <origin xyz="${chassis_length/2} 0 ${chassis_height/2}"/>
             <geometry>
-                <mesh filename="package://articubot_one/meshes/gazebo_turt_body.dae" scale="1 1 1"/>
+                <mesh filename="package://articubot_one/meshes/gazebo_turt_body.stl" scale="1 1 1"/>
             </geometry>
             <material name="orange"/>

Commit message: sdsdsd

File: description/robot_core.xacro (robot description, xacro)
@@ -6,5 +6,5 @@
     <xacro:property name="chassis_height" value="0.130"/>
     <xacro:property name="chassis_mass" value="1.0"/>
-    <xacro:property name="wheel_radius" value="0.075"/>
+    <xacro:property name="wheel_radius" value="0.0375"/>
     <xacro:property name="wheel_thickness" value="0.015"/>
     <xacro:property name="wheel_mass" value="0.05"/>

Commit message: 2343243

File: description/robot_core.xacro (robot description, xacro)
@@ -3,6 +3,6 @@
     <xacro:include filename="inertial_macros.xacro"/>
     <xacro:property name="chassis_length" value="0.220"/>
-    <xacro:property name="chassis_width" value="0.195"/>
-    <xacro:property name="chassis_height" value="0.130"/>
+    <xacro:property name="chassis_width" value="0.200"/>
+    <xacro:property name="chassis_height" value="0.150"/>
     <xacro:property name="chassis_mass" value="1.0"/>
     <xacro:property name="wheel_radius" value="0.0375"/>

Commit message: ere

File: description/robot_core.xacro (robot description, xacro)
@@ -2,9 +2,9 @@
 <robot xmlns:xacro="http://www.ros.org/wiki/xacro" >
     <xacro:include filename="inertial_macros.xacro"/>
-    <xacro:property name="chassis_length" value="0.220"/>
+    <xacro:property name="chassis_length" value="0.230"/>
     <xacro:property name="chassis_width" value="0.200"/>
     <xacro:property name="chassis_height" value="0.150"/>
     <xacro:property name="chassis_mass" value="1.0"/>
-    <xacro:property name="wheel_radius" value="0.0375"/>
+    <xacro:property name="wheel_radius" value="0.035"/>
     <xacro:property name="wheel_thickness" value="0.015"/>
     <xacro:property name="wheel_mass" value="0.05"/>

Commit message: fgoo

File: description/robot_core.xacro (robot description, xacro)
@@ -13,5 +13,5 @@
     <xacro:property name="wheel_offset_z" value="0.035"/>
     <xacro:property name="caster_wheel_radius" value="0.01"/>
-    <xacro:property name="caster_wheel_mass" value="0.01"/>
+    <xacro:property name="caster_wheel_mass" value="1"/>
     <xacro:property name="caster_wheel_offset_x" value="0.055"/>
     <xacro:property name="caster_wheel_offset_z" value="${wheel_offset_z - wheel_radius + caster_wheel_radius}"/>
@@ -59,5 +59,5 @@
             <origin xyz="${chassis_length/2} 0 ${chassis_height/2}"/>
             <geometry>
-                <box size="${chassis_length} ${chassis_width} ${chassis_height}"/>
+                <mesh filename="package://articubot_one/meshes/gazebo_turt_body.stl" scale="1 1 1"/>
             </geometry>
         </collision>

Commit message: Changes

File: description/robot_core.xacro (robot description, xacro)
@@ -38,11 +38,10 @@
         <parent link="base_link"/>
         <child link="base_footprint"/>
-        <origin xyz="0 0 0" rpy="0 0 0"/>
+        <origin xyz="0 0 0" rpy="0 0 ${pi}"/>
     </joint>
-    <link name="base_footprint">
-    </link>
+    <link name="base_footprint"/>
     <!-- CHASSIS LINK -->
     <joint name="chassis_joint" type="fixed">
-        <parent link="base_link"/>
+        <parent link="base_footprint"/>
         <child link="chassis"/>
         <origin xyz="${-wheel_offset_x} 0 ${-wheel_offset_z}"/>
@@ -107,5 +106,5 @@
                 <cylinder radius="${wheel_radius}" length="${wheel_thickness}"/>
             </geometry>
-            <material name="blue"/>
+            <material name="red"/>
         </visual>
         <collision>

Commit message: Base link

File: description/robot_core.xacro (robot description, xacro)
@@ -122,5 +122,5 @@
     <!-- CASTER WHEEL LINK -->
     <joint name="caster_wheel_joint" type="fixed">
-        <parent link="chassis"/>
+        <parent link="base_link"/>
         <child link="caster_wheel"/>
         <origin xyz="${caster_wheel_offset_x} 0 ${caster_wheel_offset_z}"/>
